Commit message: ur5 control with GSmini without tactile

File: environment/ur5_robotiq_GSmini/urdf/ur5_robotiq_GSmini.urdf (robot description, URDF)
Before this commit: robot ur5_robotiq_GSmini, 26 links, 25 joints
Links:
- removed link left_gelsight_connector
- removed link left_gelsight_mini_base_link
- removed link left_gelsight_mini_soft_link
- removed link left_inner_finger_pad
- removed link right_gelsight_connector
- removed link right_gelsight_mini_base_link
- removed link right_gelsight_mini_soft_link
- removed link right_inner_finger_pad
- link base_link: geometry collision mesh filename=../meshes/ur5/collision/base.stl; visual mesh filename=../meshes/ur5/visual/base.dae
- link forearm_link: geometry collision mesh filename=../meshes/ur5/collision/forearm.stl; visual mesh filename=../meshes/ur5/visual/forearm.dae
- link left_inner_finger: geometry collision box size=0.022 0.00635 0.0375; visual box size=0.022 0.00635 0.0375
- link left_inner_knuckle: geometry visual mesh filename=../meshes/robotiq_85/visual/robotiq_arg2f_85_inner_knuckle.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 scale=0.001 0.001 0.001
- link left_outer_finger: geometry visual mesh filename=../meshes/robotiq_85/visual/robotiq_arg2f_85_outer_finger.d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 scale=0.001 0.001 0.001
- link left_outer_knuckle: geometry visual mesh filename=../meshes/robotiq_85/visual/robotiq_arg2f_85_outer_knuckle.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 scale=0.001 0.001 0.001
- link right_inner_finger: geometry collision box size=0.022 0.00635 0.0375; visual box size=0.022 0.00635 0.0375
- link right_inner_knuckle: geometry visual mesh filename=../meshes/robotiq_85/visual/robotiq_arg2f_85_inner_knuckle.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 scale=0.001 0.001 0.001
- link right_outer_finger: geometry visual mesh filename=../meshes/robotiq_85/visual/robotiq_arg2f_85_outer_finger.d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 scale=0.001 0.001 0.001
- link right_outer_knuckle: geometry visual mesh filename=../meshes/robotiq_85/visual/robotiq_arg2f_85_outer_knuckle.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 scale=0.001 0.001 0.001
- link shoulder_link: geometry collision mesh filename=../meshes/ur5/collision/shoulder.stl; visual mesh filename=../meshes/ur5/visual/shoulder.dae
- link upper_arm_link: geometry collision mesh filename=../meshes/ur5/collision/upperarm.stl; visual mesh filename=../meshes/ur5/visual/upperarm.dae
- link wrist_1_link: geometry collision mesh filename=../meshes/ur5/collision/wrist1.stl; visual mesh filename=../meshes/ur5/visual/wrist1.dae
- link wrist_2_link: geometry collision mesh filename=../meshes/ur5/collision/wrist2.stl; visual mesh filename=../meshes/ur5/visual/wrist2.dae
- link wrist_3_link: geometry collision mesh filename=../meshes/ur5/collision/wrist3.stl; visual mesh filename=../meshes/ur5/visual/wrist3.dae
Joints:
- removed joint left_gelsight_connector_joint
- removed joint left_gelsight_mini_base_joint
- removed joint left_gelsight_mini_soft_joint
- removed joint left_inner_finger_pad_joint
- removed joint right_gelsight_connector_joint
- removed joint right_gelsight_mini_base_joint
- removed joint right_gelsight_mini_soft_joint
- removed joint right_inner_finger_pad_joint

Commit message: cube tactile grasp with GSmini and ur

File: environment/ur5_robotiq_GSmini/urdf/ur5_robotiq_GSmini.urdf (robot description, URDF)
Before this commit: robot ur5_robotiq_GSmini, 18 links, 17 joints
Links:
- added link left_gelsight_connector, mass 0.005; visual mesh filename=../meshes/gelsight_robotiq_connector/visual/Connector.stl scale=1.0 1.0 1.0
- added link left_gelsight_mini_camera, mass 0.0001
- added link left_gelsight_mini_case, mass 0.02; visual mesh filename=../meshes/gelsight_mini/visual/GSmini_base_link.stl scale=1.0 1.0 1.0
- added link left_gelsight_mini_gelpad, mass 0.003; collision box size=0.02386397 0.00525 0.02822794; visual mesh filename=../meshes/gelsight_mini/visual/GSmini_soft_link.stl scale=1.0 1.0 1.0
- added link right_gelsight_connector, mass 0.005; visual mesh filename=../meshes/gelsight_robotiq_connector/visual/Connector.stl scale=1.0 1.0 1.0
- added link right_gelsight_mini_camera, mass 0.0001
- added link right_gelsight_mini_case, mass 0.02; visual mesh filename=../meshes/gelsight_mini/visual/GSmini_base_link.stl scale=1.0 1.0 1.0
- added link right_gelsight_mini_gelpad, mass 0.003; collision box size=0.02386397 0.00525 0.02822794; visual mesh filename=../meshes/gelsight_mini/visual/GSmini_soft_link.stl scale=1.0 1.0 1.0
- link left_inner_finger: geometry collision box size=0.022 0.00635 0.0375; collision mesh filename=../meshes/robotiq_85/collision/robotiq_arg2f_85_inner_finge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 scale=0.001 0.001 0.001
- link left_inner_knuckle: geometry collision mesh filename=../meshes/robotiq_85/collision/robotiq_arg2f_85_inner_knuck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 scale=0.001 0.001 0.001; visual mesh filename=../meshes/robotiq_85/visual/robotiq_arg2f_85_inner_knuckle.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 scale=0.001 0.001 0.001
- link left_outer_finger: geometry collision mesh filename=../meshes/robotiq_85/collision/robotiq_arg2f_85_outer_finge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 scale=0.001 0.001 0.001; visual mesh filename=../meshes/robotiq_85/visual/robotiq_arg2f_85_outer_finger.d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 scale=0.001 0.001 0.001
- link left_outer_knuckle: geometry collision mesh filename=../meshes/robotiq_85/collision/robotiq_arg2f_85_outer_knuck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 scale=0.001 0.001 0.001; visual mesh filename=../meshes/robotiq_85/visual/robotiq_arg2f_85_outer_knuckle.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 scale=0.001 0.001 0.001
- link right_inner_finger: geometry collision box size=0.022 0.00635 0.0375; collision mesh filename=../meshes/robotiq_85/collision/robotiq_arg2f_85_inner_finge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 scale=0.001 0.001 0.001
- link right_inner_knuckle: geometry collision mesh filename=../meshes/robotiq_85/collision/robotiq_arg2f_85_inner_knuck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 scale=0.001 0.001 0.001; visual mesh filename=../meshes/robotiq_85/visual/robotiq_arg2f_85_inner_knuckle.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 scale=0.001 0.001 0.001
- link right_outer_finger: geometry collision mesh filename=../meshes/robotiq_85/collision/robotiq_arg2f_85_outer_finge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 scale=0.001 0.001 0.001; visual mesh filename=../meshes/robotiq_85/visual/robotiq_arg2f_85_outer_finger.d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 scale=0.001 0.001 0.001
- link right_outer_knuckle: geometry collision mesh filename=../meshes/robotiq_85/collision/robotiq_arg2f_85_outer_knuck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 scale=0.001 0.001 0.001; visual mesh filename=../meshes/robotiq_85/visual/robotiq_arg2f_85_outer_knuckle.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 scale=0.001 0.001 0.001
Joints:
- added joint left_gelsight_connector_fixed_attachment_joint: type fixed, parent left_inner_finger, child left_gelsight_connector, origin xyz=-0.001576 -0.0143493446692936 0.03242 rpy=3.141592654 0.0 3.141592654
- added joint left_gelsight_mini_camera_joint: type fixed, parent left_gelsight_mini_case, child left_gelsight_mini_camera, origin xyz=0 0 0 rpy=0 0 0
- added joint left_gelsight_mini_case_fixed_attachment_joint: type fixed, parent left_gelsight_connector, child left_gelsight_mini_case, origin xyz=0 0 0 rpy=0 0 0
- added joint left_gelsight_mini_gelpad_soft_attachment_joint: type fixed, parent left_gelsight_mini_case, child left_gelsight_mini_gelpad, origin xyz=0 0 0 rpy=0 0 0
- added joint right_gelsight_connector_fixed_attachment_joint: type fixed, parent right_inner_finger, child right_gelsight_connector, origin xyz=-0.001576 -0.0143493446692936 0.03242 rpy=3.141592654 0.0 3.141592654
- added joint right_gelsight_mini_camera_joint: type fixed, parent right_gelsight_mini_case, child right_gelsight_mini_camera, origin xyz=0 0 0 rpy=0 0 0
- added joint right_gelsight_mini_case_fixed_attachment_joint: type fixed, parent right_gelsight_connector, child right_gelsight_mini_case, origin xyz=0 0 0 rpy=0 0 0
- added joint right_gelsight_mini_gelpad_soft_attachment_joint: type fixed, parent right_gelsight_mini_case, child right_gelsight_mini_gelpad, origin xyz=0 0 0 rpy=0 0 0
