Commit message: RL training begin

File: environment/ur5_robotiq_GSmini/urdf/ur5_robotiq_GSmini_new.urdf (robot description, URDF)
Before this commit: robot ur5_robotiq_GSmini, 26 links, 25 joints
Links:
- link left_gelsight_connector: geometry collision mesh filename=../meshes/gelsight_robotiq_connector/visual/adaptor_4.STL scale=0.001 0.001 0.001; visual mesh filename=../meshes/gelsight_robotiq_connector/visual/adaptor_4.STL scale=0.001 0.001 0.001
- link right_gelsight_connector: geometry collision mesh filename=../meshes/gelsight_robotiq_connector/visual/adaptor_4.STL scale=0.001 0.001 0.001; visual mesh filename=../meshes/gelsight_robotiq_connector/visual/adaptor_4.STL scale=0.001 0.001 0.001
Joints:
- joint left_gelsight_connector_fixed_attachment_joint: origin xyz=-0.001576 -0.0093293446692936 0.03532 rpy=3.141592654 0.0 3.141592654 -> xyz=-0.001576 -0.0073293446692936 0.03532 rpy=3.141592654 0.0 3.141592654
- joint left_gelsight_mini_case_fixed_attachment_joint: origin xyz=0 0.0085 0 rpy=0 0 0 -> xyz=0 0.0075 0 rpy=0 0 0
- joint right_gelsight_connector_fixed_attachment_joint: origin xyz=-0.001576 -0.0093293446692936 0.03532 rpy=3.141592654 0.0 3.141592654 -> xyz=-0.001576 -0.0073293446692936 0.03532 rpy=3.141592654 0.0 3.141592654
- joint right_gelsight_mini_case_fixed_attachment_joint: origin xyz=0 0.0085 0 rpy=0 0 0 -> xyz=0 0.0075 0 rpy=0 0 0
